Commit message: enabling dual-arm

File: hiro_common/urdf/hiro.urdf.xacro (robot description, xacro)
@@ -12,6 +12,6 @@
 	<xacro:head />
   <xacro:arm side="r" reflect="1" />
-  <xacro:hand side="r" reflect="1" />
+  <xacro:hand side="r" reflect="1" reflect2="0" />
   <xacro:arm side="l" reflect="-1" />
-  <xacro:hand side="l" reflect="-1" />
+  <xacro:hand side="l" reflect="-1" reflect2="1" />
 </robot>

File: hiro_common/urdf/hiro_hand.urdf.xacro (robot description, xacro)
@@ -1,10 +1,10 @@
 <?xml version="1.0"?>
 <robot xmlns:xacro="http://www.ros.org/wiki/xacro" name="hiro_hand">
-  <xacro:macro name="hand" params="side reflect">
+  <xacro:macro name="hand" params="side reflect reflect2">
 	  <joint name="joint_${side}hand_palm" type="fixed">
 		  <parent link="link_${side}wrist_roll"/>
 		  <child link="link_${side}hand_palm"/>
 		  <!--origin xyz="${(-1*(0.130/2))+(-1*(0.010/2))} ${(-1*(0.055/2))+(-1*(0.035/2))} 0" rpy="0 0 0"/-->
-		  <origin xyz="${-1*((0.130/2)+(0.010/2))} ${reflect*-1*((0.055/2)+(0.035/2))} 0" rpy="0 0 0"/>
+		  <origin xyz="${-1*((0.130/2)+(0.010/2))} ${reflect*-1*((0.055/2)+(0.035/2))} 0" rpy="0 0 ${reflect2*M_PI}"/>
 		  <!--
 		    Origin x is shifted a half of x-dimension of hand_palm plus a half of x-dimension of link_${side}wrist_roll in the appropriate direction

Commit message: fix joint limit values in wrist_yaw joint

File: hiro_common/urdf/hiro.urdf.xacro (robot description, xacro)
@@ -11,7 +11,7 @@
 	<xacro:chest />
 	<xacro:head />
-  <xacro:arm side="r" reflect="1" />
+  <xacro:arm side="r" reflect="1" reflect2="0" />
   <xacro:hand side="r" reflect="1" reflect2="0" />
-  <xacro:arm side="l" reflect="-1" />
+  <xacro:arm side="l" reflect="-1" reflect2="1" />
   <xacro:hand side="l" reflect="-1" reflect2="1" />
 </robot>

File: hiro_common/urdf/hiro_arm.urdf.xacro (robot description, xacro)
@@ -3,5 +3,5 @@
   <!-- TODO Find out the exact value for below-->
   <xacro:property name="dist_to_wrist_pitch_mesh_boundary" value="-0.025" />
-  <xacro:macro name="arm" params="side reflect">
+  <xacro:macro name="arm" params="side reflect reflect2">
   	<joint name="joint_${side}shoulder_yaw" type="revolute">
       <parent link="link_chest_yaw"/>
@@ -114,5 +114,5 @@
       <origin xyz="-0.02 0.0 -0.22" rpy="0 0 0"/>
       <axis xyz="0 0 1"/>
-      <limit lower="${-195*rad_per_deg}" upper="${135*rad_per_deg}" effort="1000.0" velocity="0.5"/>
+      <limit lower="${(-195+reflect2*60)*rad_per_deg}" upper="${(135+reflect2*60)*rad_per_deg}" effort="1000.0" velocity="0.5"/>
       <!--safety_controller  soft_lower_limit="${-190*rad_per_deg}" soft_upper_limit="${130*rad_per_deg}" k_position="0" k_velocity="0" /-->
       <!-- rotorInertia	3.74e-03 -->
